File: Browse/t1.kicad_pcb (KiCad board)
At the start: 4 copper layers, 63 x 35.6 mm, 47 parts, among them J1 Barrel_Jack_Switch, J2 USB_B, J3 P1, J4 2x2M, J5 ICSP1, J6 P2, U1 ATmega8U2-AU, Y1 16MHz

Commit message: Deploying to main from @ set-soft/kibot_variants_arduprog_test@f2b5671748de411d028c9745b59ca051d219371f 🚀
Connections:
- U1 pad 14: Net-(U1-Pad14) -> unconnected-(U1-PB0-Pad14)
