File: Browse/t1.kicad_sch (KiCad schematic)
At the start: 47 parts, among them J1 Barrel_Jack_Switch, J2 USB_B, J3 P1, J4 2x2M, J5 ICSP1, J6 P2, U1 ATmega8U2-AU, Y1 16MHz

Commit message: Deploying to main from @ set-soft/kibot_variants_arduprog_test@3a250a0e673ff2005b39d0bb688751c13561674d 🚀
Parts:
- J3: symbol Connector:Conn_01x05_Male -> Connector:Conn_01x05_Pin
- J6: symbol Connector:Conn_01x06_Male -> Connector:Conn_01x06_Pin
