File: Browse/t1.kicad_sch (KiCad schematic)
At the start: 47 parts, among them J1 Barrel_Jack_Switch, J2 USB_B, J3 P1, J4 2x2M, J5 ICSP1, J6 P2, U1 ATmega8U2-AU, Y1 16MHz

Commit message: Deploying to main from @ set-soft/kibot_variants_arduprog_test@135d77b440a929b8dc4f6d317a81e03ec03b4d04 🚀
Connections:
- net at FB1.1, VR1.2, VR2.2: now also J2.SH (Shield); no longer J2.5 (Shield)
